File: MM1_FLASH_128k_A.sch (KiCad schematic (older format))
At the start: 6 parts, among them J1 MM1_edgeConnector_5530843-2, U1 SST39LF010-55-4C-NH

Commit message: materials, images
Parts:
- JP1: footprint TestPoint:TestPoint_2Pads_Pitch2.54mm_Drill0.8mm -> Connector_PinHeader_2.54mm:PinHeader_1x02_P2.54mm_Vertical
Changed lines of the file:
@@
 F 0 "JP1" H 4200 3935 50  0000 C CNN
 F 1 "Jumper_2_Open" H 4200 3844 50  0000 C CNN
-F 2 "TestPoint:TestPoint_2Pads_Pitch2.54mm_Drill0.8mm" H 4200 3700 50  0001 C CNN
+F 2 "Connector_PinHeader_2.54mm:PinHeader_1x02_P2.54mm_Vertical" H 4200 3700 50  0001 C CNN
 F 3 "~" H 4200 3700 50  0001 C CNN
 	1    4200 3700
