File: MM1_FLASH_128k_A.kicad_pcb (KiCad board)
At the start: 2 copper layers, 51.5 x 34 mm, 6 parts, among them J1 MM1_edgeConnector_5530843-2, U1 SST39LF010-55-4C-NH

Commit message: materials, images
Parts:
- JP1: footprint TestPoint:TestPoint_2Pads_Pitch2.54mm_Drill0.8mm -> Connector_PinHeader_2.54mm:PinHeader_1x02_P2.54mm_Vertical
- turned JP1 to 0 degrees
Routing:
- net /MEM_~CE: track 50.7 -> 52.0 mm
- net /MEM_~WE: track 34.7 -> 36.0 mm

Commit message: Gerbert
Other:
- net class Power added: clearance 0.2, trace_width 0.25, via_dia 0.45, via_drill 0.2
- net class Tension removed
- rule pad_to_mask_clearance: 0.2 -> 0
